File: pcb/keypad/keypad.kicad_pcb (KiCad board)
At the start: 2 copper layers, 81 x 64.3 mm, 9 parts, among them J1 OLED_DISPLAY, SW1 SW_Push, SW2 SW_Push, SW3 SW_Push, SW4 SW_Push, SW5 RotaryEncoder_Switch, U1 XIAO-RP2040-DIP

Commit message: Fix error in pcb
Connections:
- U1 pad 12: Net-(D2-DIN) -> unconnected-(U1-3V3-Pad12)
- U1 pad 7: unconnected-(U1-GPIO0/TX-Pad7) -> Net-(D2-DIN)
Routing:
- net Net-(D2-DIN): track 38.5 -> 20.4 mm
Changed lines of the file:
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@@
 	(net 14 "Net-(U1-GPIO29{slash}ADC3{slash}A3)")
 	(net 15 "Net-(U1-GPIO26{slash}ADC0{slash}A0)")
-	(net 16 "unconnected-(U1-GPIO0{slash}TX-Pad7)")
+	(net 16 "unconnected-(U1-3V3-Pad12)")
 	(footprint "Rotary_Encoder:RotaryEncoder_Alps_EC11E-Switch_Vertical_H20mm"
 		(layer "F.Cu")
@@
 		(property ki_fp_filters "RotaryEncoder*Switch*")
 		(sheetname "/")
-		(sheetfile "Tastierino.kicad_sch")
+		(sheetfile "keypad.kicad_sch")
 		(attr through_hole)
 		(fp_line
@@
 		(property ki_fp_filters "Connector*:*_1x??_*")
 		(sheetname "/")
-		(sheetfile "Tastierino.kicad_sch")
+		(sheetfile "keypad.kicad_sch")
 		(attr through_hole)
 		(fp_line
@@
 		)
 		(sheetname "/")
-		(sheetfile "Tastierino.kicad_sch")
+		(sheetfile "keypad.kicad_sch")
 		(attr through_hole)
 		(fp_line
@@
 		)
 		(sheetname "/")
-		(sheetfile "Tastierino.kicad_sch")
+		(sheetfile "keypad.kicad_sch")
 		(attr through_hole)
 		(fp_line
@@
 		)
 		(sheetname "/")
-		(sheetfile "Tastierino.kicad_sch")
+		(sheetfile "keypad.kicad_sch")
 		(attr through_hole)
 		(fp_line
@@
 		(property ki_fp_filters "LED*SK6812*PLCC*5.0x5.0mm*P3.2mm*")
 		(sheetname "/")
-		(sheetfile "Tastierino.kicad_sch")
+		(sheetfile "keypad.kicad_sch")
 		(attr smd)
 		(fp_line
@@
 		)
 		(sheetname "/")
-		(sheetfile "Tastierino.kicad_sch")
+		(sheetfile "keypad.kicad_sch")
 		(attr through_hole)
 		(fp_line
@@
 		)
 		(sheetname "/")
-		(sheetfile "Tastierino.kicad_sch")
+		(sheetfile "keypad.kicad_sch")
 		(attr smd)
 		(fp_line
@@
 			(layers "F.Cu" "F.Mask")
 			(roundrect_rratio 0.1)
-			(net 16 "unconnected-(U1-GPIO0{slash}TX-Pad7)")
+			(net 5 "Net-(D2-DIN)")
 			(pinfunction "GPIO0/TX")
 			(pintype "passive")
@@
 			(layers "*.Cu" "*.Mask")
 			(remove_unused_layers no)
-			(net 16 "unconnected-(U1-GPIO0{slash}TX-Pad7)")
+			(net 5 "Net-(D2-DIN)")
 			(pinfunction "GPIO0/TX")
 			(pintype "passive")
@@
 			(layers "*.Cu" "*.Mask")
 			(remove_unused_layers no)
-			(net 5 "Net-(D2-DIN)")
+			(net 16 "unconnected-(U1-3V3-Pad12)")
 			(pinfunction "3V3")
 			(pintype "passive")
@@
 			(layers "F.Cu" "F.Mask")
 			(roundrect_rratio 0.1)
-			(net 5 "Net-(D2-DIN)")
+			(net 16 "unconnected-(U1-3V3-Pad12)")
 			(pinfunction "3V3")
 			(pintype "passive")
@@
 		(property ki_fp_filters "LED*SK6812*PLCC*5.0x5.0mm*P3.2mm*")
 		(sheetname "/")
-		(sheetfile "Tastierino.kicad_sch")
+		(sheetfile "keypad.kicad_sch")
 		(attr smd)
 		(fp_line
@@
 	)
 	(segment
+		(start 137.63625 102.33375)
+		(end 135.67 104.3)
+		(width 0.2)
+		(layer "F.Cu")
+		(net 5)
+	)
+	(segment
 		(start 125.0875 101.1575)
 		(end 125.0875 97.63125)
@@
 	)
 	(segment
-		(start 138.55625 104.3)
-		(end 152.87625 89.98)
+		(start 137.63625 100.14)
+		(end 137.63625 102.33375)
 		(width 0.2)
 		(layer "F.Cu")
@@
 	)
 	(segment
-		(start 126.09 102.16)
-		(end 125.0875 101.1575)
+		(start 135.67 104.3)
+		(end 134.2 104.3)
 		(width 0.2)
 		(layer "F.Cu")
@@
 	)
 	(segment
-		(start 134.2 104.3)
-		(end 138.55625 104.3)
+		(start 126.09 102.16)
+		(end 125.0875 101.1575)
 		(width 0.2)
 		(layer "F.Cu")
