File: pcb/keypad/keypad.kicad_sch (KiCad schematic)
At the start: 9 parts, among them J1 OLED_DISPLAY, SW1 SW_Push, SW2 SW_Push, SW3 SW_Push, SW4 SW_Push, SW5 RotaryEncoder_Switch, U1 XIAO-RP2040-DIP

Commit message: Fix error in pcb
Connections:
- net at D2.2 (DIN): now also U1.7 (GPIO0/TX); no longer U1.12 (3V3)
Changed lines of the file:
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@@
+	(wire
+		(pts
+			(xy 127 121.92) (xy 129.54 121.92)
+		)
+		(stroke
+			(width 0)
+			(type default)
+		)
+	)
 	(wire
 		(pts
@@
 	(wire
 		(pts
+			(xy 127 43.18) (xy 127 121.92)
+		)
+		(stroke
+			(width 0)
+			(type default)
+		)
+	)
+	(wire
+		(pts
 			(xy 179.07 156.21) (xy 179.07 114.3)
 		)
@@
 	(wire
 		(pts
-			(xy 182.88 69.85) (xy 172.72 69.85)
-		)
-		(stroke
-			(width 0)
-			(type default)
-		)
-	)
-	(wire
-		(pts
 			(xy 184.15 57.15) (xy 184.15 50.8)
 		)
@@
 	(wire
 		(pts
-			(xy 172.72 43.18) (xy 176.53 43.18)
-		)
-		(stroke
-			(width 0)
-			(type default)
-		)
-	)
-	(wire
-		(pts
 			(xy 85.09 106.68) (xy 129.54 106.68)
 		)
@@
 	(wire
 		(pts
-			(xy 182.88 106.68) (xy 182.88 69.85)
-		)
-		(stroke
-			(width 0)
-			(type default)
-		)
-	)
-	(wire
-		(pts
 			(xy 118.11 40.64) (xy 118.11 99.06)
 		)
@@
 	(wire
 		(pts
-			(xy 172.72 69.85) (xy 172.72 43.18)
-		)
-		(stroke
-			(width 0)
-			(type default)
-		)
-	)
-	(wire
-		(pts
 			(xy 218.44 29.21) (xy 184.15 29.21)
 		)
@@
 	(wire
 		(pts
+			(xy 176.53 43.18) (xy 127 43.18)
+		)
+		(stroke
+			(width 0)
+			(type default)
+		)
+	)
+	(wire
+		(pts
 			(xy 73.66 43.18) (xy 73.66 50.8)
 		)
 		(stroke
-			(width 0)
-			(type default)
-		)
-	)
-	(wire
-		(pts
-			(xy 165.1 106.68) (xy 182.88 106.68)
-		)
-		(stroke
